File: Pomiar czasu/eagle/master - Copy.brd (EAGLE design)
At the start: 246.4 x 107.9 mm, 102 parts, among them IC1 MEGA8-AI, IC2 lf33, IC3 MEGA8-AI, IC4 lf33, U1 RFM69HW, U2 RFM69HW

Commit message: RFM69:communication master->sensor works!
Parts:
- added R41: 470, rcl:R0805
- added R42: 220, rcl:R0805
- added R43, R44: 0R, rcl:R1206
- R20, R21: value 10k -> 0R; device rcl:R0805 -> rcl:R1206
- R22, R23: value 220 -> 10k
- R26, R27: value 15R -> 220
- R29, R31: value 470 -> 15R
- R40: value 220 -> 470
- moved R20 109.7 mm to (91.1, 31.1), turned to 0 degrees
- moved R21 78.3 mm to (91.1, 23.5), flipped to the top, turned to 0 degrees
- moved R27 69.9 mm to (144.5, 23.5), flipped to the bottom, turned to 0 degrees
- moved R29 67.4 mm to (188.9, 92.7), flipped to the top
- moved R28 64.0 mm to (186.4, 77.5), turned to 270 degrees
- moved R26 62.4 mm to (144.5, 26.0), flipped to the bottom, turned to 0 degrees
- moved R22 58.4 mm to (198.4, 55.2), flipped to the top, turned to 180 degrees
- moved R35 55.1 mm to (180.7, 25.4), flipped to the bottom
- moved R40 54.3 mm to (191.5, 77.5), turned to 90 degrees
- moved R36 52.3 mm to (190.8, 25.4), flipped to the bottom
- moved S2 39.1 mm to (158.8, 66.4)
- moved S1 39.1 mm to (87.9, 66.4)
- moved R23 29.2 mm to (165.7, 48.3), turned to 90 degrees
- moved R31 23.2 mm to (209.9, 17.8), flipped to the top
- moved R30 20.6 mm to (57.8, 92.7)
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Connections:
- removed net N$50: R35.1, SV3.4
- removed net N$51: R36.1, SV3.2
- removed net N$52: R37.2, SV3.5
- removed net N$53: R38.2, SV3.3
- removed net N$54: R39.2, SV3.1
- removed net N$55: R40.2, USART1.1
- new net LED_FALSTART_GND: Q4.3, SV1.8
- new net LED_FALSTART_GND1: Q2.3, SV3.8
- new net LED_GO_GND: Q3.3, SV1.9
- new net LED_GO_GND1: Q1.3, SV3.9
- new net N$57: D10.C, R24.1, R43.2
- new net N$58: D7.C, R27.1, R44.2
- new net N$59: S2.1, U1.15
- new net N$60: S2.4, U1.12
- new net N$61: S2.3, U1.13
- new net N$62: S2.2, U1.14
- net +3V1: now also R22.1, R23.1, R28.2, R29.2; no longer R20.1, R21.1, R26.2, R27.2
- net GND: now also Q3.2, Q4.2; no longer SV1.8, SV1.9
- net GND1: now also Q1.2, Q2.2, R31.2; no longer R28.2, SV3.8, SV3.9
- net LED_FALSTART: now also R30.1; no longer Q4.2
- net LED_FALSTART1: now also R29.1; no longer Q2.2
- net LED_GO: now also R2.1; no longer Q3.2
- net LED_GO1: now also R28.1; no longer Q1.2
- net LED_S10: now also R32.2; no longer R29.2
- net LED_S6: now also R36.1; no longer R34.1
- net LED_S7: now also R35.1; no longer R33.1
- net LED_S8: now also R34.1; no longer R32.1
- net LED_S9: now also R33.2; no longer R31.2
- net LED_Y10: now also R39.1; no longer R37.1
- net LED_Y6: now also R41.1; no longer R39.1
- net LED_Y7: now also R38.2; no longer R36.2
- net LED_Y8: now also R40.1; no longer R38.1
- net LED_Y9: now also R37.2; no longer R35.2
- net MISO: now also R21.1, S1.6; no longer S1.8, U2.13
- net MISO1: now also R44.1, S2.6; no longer S2.8, U1.13
- net MOSI: now also R20.1, S1.7; no longer S1.5, U2.14
- net MOSI1: now also R43.1, S2.7; no longer S2.5, U1.14
- net N$1: now also D1.C, R11.1, R21.2; no longer Q3.3, R2.1
- net N$10: now also S1.4, U2.12; no longer D3.C, R9.1, S1.3
- net N$11: now also S1.3, U2.13; no longer D2.C, R10.1, S1.2
- net N$12: now also S1.2, U2.14; no longer D1.C, R11.1, S1.1
- net N$2: now also D4.C, R20.2, R8.1; no longer Q4.3, R30.1
- net N$32: now also R23.2; no longer R21.2
- net N$34: now also R24.2, U$4.1; no longer D10.C, R22.1, S2.4
- net N$35: now also R27.2, U$4.9; no longer D9.C, R23.1, S2.3
- net N$36: now also R26.2, U$4.7; no longer D8.C, R24.1, S2.2
- net N$37: now also R25.2, U$4.5; no longer D7.C, R25.1, S2.1
- net N$38: now also LED_RED1.1, R31.1; no longer R22.2, U$4.1
- net N$39: now also R32.1, SV4.4; no longer R25.2, U$4.9
- net N$40: now also R33.1, SV4.2; no longer R24.2, U$4.7
- net N$41: now also R34.2, SV4.5; no longer R23.2, U$4.5
- net N$42: now also R35.2, SV4.3; no longer Q1.3, R26.1
- net N$43: now also R36.2, SV4.1; no longer Q2.3, R27.1
- net N$44: now also R37.1, SV3.4; no longer LED_RED1.1, R28.1
- net N$45: now also R38.1, SV3.2; no longer R29.1, SV4.4
- net N$46: now also R39.2, SV3.5; no longer R31.1, SV4.2
- net N$47: now also R40.2, SV3.3; no longer R32.2, SV4.5
- net N$48: now also R41.2, SV3.1; no longer R33.2, SV4.3
- net N$49: now also R42.2, USART1.1; no longer R34.2, SV4.1
- net N$8: now also S1.1, U2.15; no longer D4.C, R8.1, S1.4
- net RESET: now also D3.C, R9.1; no longer S1.6
- net RESET1: now also D9.C, R22.2, R25.1; no longer R20.2, S2.6
- net RX1: now also R42.1; no longer R40.1
- net SCK: now also D2.C, R10.1, S1.5; no longer S1.7, U2.12
- net SCK1: now also D8.C, R26.1, S2.5; no longer S2.7, U1.12
- net SS: now also S1.8; no longer U2.15
- net SS1: now also S2.8; no longer U1.15
Routing:
- net N$60: track 0.00 -> 39.3 mm
- net +3V3: track 173.9 -> 209.5 mm
- net +3V1: track 173.9 -> 209.5 mm
- net N$61: track 0.00 -> 33.6 mm
- net N$42: track 2.12 -> 30.8 mm, vias 0 -> 1
- net N$62: track 0.00 -> 27.9 mm
- net N$48: track 30.8 -> 6.03 mm, vias 1 -> 0
- net N$10: track 16.2 -> 39.3 mm
- net RESET: track 71.6 -> 93.9 mm
- net RESET1: track 71.6 -> 93.9 mm
- net N$59: track 0.00 -> 21.2 mm
- net MOSI: track 94.6 -> 115.2 mm
- net MOSI1: track 94.6 -> 115.2 mm
- net N$50: track 20.0 -> 0.00 mm
- net N$58: track 0.00 -> 18.4 mm
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- added copper zone on layer 1, net N$38
- added copper zone on layer 1, net N$50
- added copper zone on layer 16, net N$51
- added copper zone on layer 16, net N$52
- added copper zone on layer 16, net N$53
- added copper zone on layer 16, net N$54
- added copper zone on layer 16, net N$55
- added copper zone on layer 1, net N$8
- removed copper zone on layer 1, net N$44
- removed copper zone on layer 16, net N$57
- removed copper zone on layer 16, net N$58
- removed copper zone on layer 16, net N$60
- removed copper zone on layer 16, net N$61
- removed copper zone on layer 1, net N$62
Other:
- board size 246.4 x 107.9 mm -> 246.7 x 107.9 mm
