File: Pomiar czasu/eagle/transceiver (2) - Copy.brd (EAGLE design)
At the start: 229.9 x 132 mm, 292 parts, among them IC1 MEGA8-AI, IC10 MEGA8-AI, IC11 LF33, IC12 LF50, IC2 LF33, IC3 LF50, IC4 MEGA8-AI, IC5 LF33, IC6 LF50, IC7 MEGA8-AI, IC8 LF33, IC9 LF50, U1 RFM69HW, U2 RFM69HW, U3 RFM69HW, U4 RFM69HW

Commit message: final v1.0
Parts:
- removed R121, R122, R123, R124, R125, R126, R127, R128: 0R, rcl:R1206
- added D25, D26, D27, D28: (no value), diode:SOD80C
- D13, D14, D19, D20, D7: value BAS16HT1G -> (none); device SparkFun:SOD-323 -> diode:SOD80C
- D15, D16, D22, D23, D9: value (none) -> BAS16HT1G; device diode:SOD80C -> SparkFun:SOD-323
- R1, R26: value 36,5R -> 330k
- R100: value 330k -> 1,2k
- R101, R27, R34, R36, R37, R66, R67, R68, R69, R98, R99: value 330k -> 1.2k
- R102, R104, R105, R106, R42, R44, R72, R74, R76: value 1.2k -> 10k
- R103, R73: value 1.2k -> 3,6k
- R107, R75: value 1,2k -> 10k
- R108: value 1.2k -> (none)
- R110: value 3,6k -> 0R; device resistor:R0805 -> rcl:R1206
- R111, R112, R52, R81, R82: value 10k -> 220R
- R113, R114, R116, R50, R80, R84: value 10k -> 0R; device resistor:R0805 -> rcl:R1206
- R115, R83: value (none) -> 0R; device resistor:R0805 -> rcl:R1206
- R118, R54, R86: value 330k -> 0R; device resistor:R0805 -> rcl:R1206
- R119, R55, R87: value 220R -> 0R; device resistor:R0805 -> rcl:R1206
- R120, R56, R88: value 820k -> 0R; device resistor:R0805 -> rcl:R1206
- R23: value 820k -> 330k
- R39, R70: value 1.2k -> 1,2k
- R40: value 1.2k -> 220R
- R43: value 1,2k -> 3,6k
- R46: value 3,6k -> 10k
- R48: value 10k -> (none)
- R51: value (none) -> 220R
- R61, R62, R63, R64, R91, R92, R93, R94: value 0R -> 330k; device rcl:R1206 -> resistor:R0805
- R65, R97: value 36,5R -> 1.2k
- R78: value 3,6k -> (none)
- R95, R96: value 0R -> 1.2k; device rcl:R1206 -> resistor:R0805
- moved R40 154.8 mm to (14.0, 27.6), flipped to the top, turned to 0 degrees
- moved D14 147.5 mm to (212.6, 25.6), flipped to the bottom, turned to 0 degrees
- moved R96 144.3 mm to (165.4, 107.3), flipped to the bottom, turned to 90 degrees
- moved R64 140.5 mm to (80.3, 82.2), flipped to the top, turned to 90 degrees
- moved R95 139.3 mm to (162.9, 107.3), flipped to the bottom, turned to 90 degrees
- moved R63 125.9 mm to (93.0, 82.5), flipped to the top, turned to 90 degrees
- moved R22 123.0 mm to (136.2, 14.3), turned to 90 degrees
- moved D7 120.6 mm to (17.3, 25.6), flipped to the top, turned to 0 degrees
- moved R23 119.3 mm to (136.8, 14.0), flipped to the bottom
- moved R94 117.4 mm to (149.5, 82.2)
- moved D13 116.7 mm to (145.4, 15.2), flipped to the bottom, turned to 0 degrees
- moved D21 112.0 mm to (17.3, 94.1), flipped to the top
- moved R93 111.7 mm to (136.8, 82.5), turned to 90 degrees
- moved R62 109.9 mm to (93.7, 82.9), flipped to the bottom
- moved R61 108.0 mm to (100.6, 85.4), turned to 180 degrees
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Connections:
- removed net N$105: R79.1, R92.2, SV6.2
- removed net N$106 (its old number): R80.1, R93.2, SV6.4
- removed net N$107 (its old number): R93.1, R94.2
- removed net N$118 (its old number): R101.1, U$14.9
- removed net N$119 (its old number): R114.1, U4.1
- removed net N$120 (its old number): C49.1, C51.1, C57.+, C59.+, D19.1, D20.1, IC11.1, IC12.1, R109.2, X4.1
- removed net N$128: R106.2, SV7.5
- removed net N$129 (its old number): R107.2, SV7.6
- removed net N$130 (its old number): R108.2, SV7.8
- removed net N$142: R121.2, R123.1
- removed net N$143 (its old number): R111.1, R124.2, SV8.2
- removed net N$144 (its old number): R112.1, R125.2, SV8.4
- removed net N$145 (its old number): R125.1, R126.2
- removed net N$151: R127.2, R128.1
- removed net N$152: R128.2, U4.2
- removed net N$43 (its old number): C25.+, C27.+, C5.1, C8.1, D7.1, D8.1, IC5.1, IC6.1, R45.2, X2.1
- removed net N$54: R44.2, SV1.8
- removed net N$57 (its old number): JP2.TIP, R26.1
- removed net N$68: R48.1, R61.2, SV4.4
- removed net N$69 (its old number): R61.1, R62.2
- removed net N$81 (its old number): R82.1, U3.1
- removed net N$82 (its old number): C33.1, C35.1, C41.+, C43.+, D13.1, D14.1, IC8.1, IC9.1, R77.2, X3.1
- removed net N$91: R75.2, SV5.6
- removed net N$92 (its old number): R76.2, SV5.8
- new net N$110: R89.2, R90.1
- new net N$111: R90.2, U3.2
- new net N$112: R91.1, U$14.1
- new net N$121: R95.2, SV7.1
- new net N$122: R96.2, SV7.2
- new net N$123: R97.2, SV7.3
- new net N$132: JP8.TIP, R108.1
- new net N$134: C55.1, C62.+, R112.1, TSOP3.V+
- new net N$135: R104.2, R105.2, R106.2, R110.1
- new net N$147: R119.2, R120.1
- new net N$148: R120.2, U4.2
- new net N$47: R27.2, SV1.1
- new net N$58: JP4.TIP, R48.1
- new net N$59: R51.1, TSOP1.OUT
- new net N$73: R59.2, R60.1
- new net N$74: R60.2, U2.2
- new net N$84: R65.2, SV5.1
- new net N$85: R66.2, SV5.2
- new net N$96: R81.1, TSOP2.OUT
- new net N$97: C39.1, C46.+, R82.1, TSOP2.V+
- net +3V1: now also D9.2, R47.2, R49.2; no longer D8.2, R52.2, R53.2
- net +3V2: now also D16.2, R77.2, R79.2, R80.2; no longer D14.2, R82.2, R84.2, R85.2
- net +3V4: now also D23.2, R107.2, R109.2, R110.2; no longer D20.2, R114.2, R116.2, R117.2
- net +5V: now also JP1.TIP; no longer R1.2
- net +5V1: now also D8.2, JP2.TIP, R48.2, R52.2; no longer D7.2, R26.2, R51.2, R55.2
- net +5V2: now also D15.2, JP5.TIP, R78.2, R82.2; no longer D13.2, R65.2, R83.2, R87.2
- net +5V3: now also D22.2, JP7.TIP, R108.2, R112.2; no longer D19.2, R115.2, R119.2, R97.2
- net ADC1: now also R42.1, R43.2; no longer R45.1, R46.2
- net ADC2: now also R72.1, R73.2; no longer R77.1, R78.2
- net ADC3: now also R102.1, R103.2; no longer R109.1, R110.2
- net DIO1: now also R59.1; no longer R63.1
- net DIO2: now also R89.1; no longer R95.1
- net DIO3: now also R119.1; no longer R127.1
- net GND: now also D7.A; no longer R23.1
- net GND1: now also D13.A, D14.A, R43.1; no longer D9.A, R46.1, R56.1
- net GND2: now also D19.A, D20.A, D21.A, R73.1; no longer D15.A, D16.A, R78.1, R88.1
- net GND3: now also D25.A, D26.A, D27.A, D28.A, R103.1; no longer D21.A, D22.A, D23.A, R110.1, R120.1
- net LED10: now also R38.1; no longer R42.1
- net LED11: now also R65.1; no longer R70.1
- net LED12: now also R66.1; no longer R71.1
- net LED13: now also R67.1; no longer R72.1
- net LED14: now also R68.1; no longer R73.1
- net LED15: now also R69.1; no longer R74.1
- net LED16: now also R95.1; no longer R102.1
- net LED17: now also R96.1; no longer R103.1
- net LED18: now also R97.1; no longer R104.1
- net LED19: now also R98.1; no longer R105.1
- net LED20: now also R99.1; no longer R106.1
- net LED6: now also R27.1; no longer R38.1
- net LED7: now also R34.1; no longer R39.1
- net LED8: now also R36.1; no longer R40.1
- net LED9: now also R37.1; no longer R41.1
- net LED_BATT_GR1: now also R39.1; no longer R43.1
- net LED_BATT_GR2: now also R70.1; no longer R75.1
- net LED_BATT_GR3: now also R100.1; no longer R107.1
- net LED_BATT_RED1: now also R41.1; no longer R44.1
- net LED_BATT_RED2: now also R71.1; no longer R76.1
- net LED_BATT_RED3: now also R101.1; no longer R108.1
- net MISO1: now also R54.2; no longer R58.2
- net MISO2: now also R84.2; no longer R90.2
- net MISO3: now also R114.2; no longer R122.2
- net MOSI1: now also R55.2; no longer R59.2
- net MOSI2: now also R85.2; no longer R91.2
- net MOSI3: now also R115.2; no longer R123.2
- net N$1: now also R40.1; no longer R22.1
- net N$100: now also D20.C, R64.2, R84.1; no longer C39.1, C46.+, R87.1, TSOP2.V+
- net N$101: now also R83.2; no longer R79.2, R80.2, R81.2
- net N$102: now also R74.1, R86.2, SV6.2; no longer D15.C, R66.2, R89.1
- net N$103: now also R75.1, R87.2, SV6.4; no longer D18.C, R69.2, R90.1
- net N$104: now also R87.1, R88.2; no longer R89.2, R91.1
- net N$113: now also R92.1, U$14.5; no longer R95.2, R96.1
- net N$114: now also R93.1, U$14.7; no longer R96.2, U3.2
- net N$115: now also R94.1, U$14.9; no longer R98.1, U$14.1
- net N$116: now also R107.1, U4.1; no longer R99.1, U$14.5
- net N$117: now also C49.1, C51.1, C57.+, C59.+, D22.1, D23.1, IC11.1, IC12.1, R102.2, X4.1; no longer R100.1, U$14.7
- net N$124: now also R98.2, SV7.4; no longer R102.2, SV7.1
- net N$125: now also R99.2, SV7.5; no longer R103.2, SV7.2
- net N$126: now also R100.2, SV7.6; no longer R104.2, SV7.3
- net N$127: now also R101.2, SV7.8; no longer R105.2, SV7.4
- net N$133: now also R111.1, TSOP3.OUT; no longer JP7.TIP, R97.1
- net N$136: now also D24.C, R113.1, R91.2; no longer JP8.TIP, R115.1
- net N$137: now also D27.C, R114.1, R94.2; no longer R118.1, TSOP3.OUT
- net N$138: now also R113.2, R115.1; no longer C55.1, C62.+, R119.1, TSOP3.V+
- net N$139: now also R104.1, R116.2, SV8.2; no longer R111.2, R112.2, R113.2, R117.1
- net N$140: now also R105.1, R117.2, SV8.4; no longer D21.C, R121.1, R98.2
- net N$141: now also R117.1, R118.2; no longer D24.C, R101.2, R122.1
- net N$22: now also R23.1, U$6.7; no longer R34.1, U$6.5
- net N$3: now also R1.1; no longer R27.1
- net N$40: now also R26.1, U$6.9; no longer R36.1, U$6.7
- net N$41: now also R47.1, U2.1; no longer R37.1, U$6.9
- net N$42: now also C25.+, C27.+, C5.1, C8.1, D8.1, D9.1, IC5.1, IC6.1, R42.2, X2.1; no longer R50.1, U2.1
- net N$48: now also R34.2, SV1.2; no longer R38.2, SV1.1
- net N$49: now also R36.2, SV1.3; no longer R39.2, SV1.2
- net N$50: now also R37.2, SV1.4; no longer R40.2, SV1.3
- net N$51: now also R38.2, SV1.5; no longer R41.2, SV1.4
- net N$52: now also R39.2, SV1.6; no longer R42.2, SV1.5
- net N$53: now also R41.2, SV1.8; no longer R43.2, SV1.6
- net N$60: now also C23.1, C30.+, R52.1, TSOP1.V+; no longer JP4.TIP, R51.1
- net N$61: now also R44.2, R45.2, R46.2, R50.1; no longer R54.1, TSOP1.OUT
- net N$62: now also D10.C, R1.2, R53.1; no longer C23.1, C30.+, R55.1, TSOP1.V+
- net N$63: now also D13.C, R26.2, R54.1; no longer R47.2, R48.2, R49.2, R53.1
- net N$64: now also R53.2, R55.1; no longer D9.C, R27.2, R57.1
- net N$65: now also R44.1, R56.2, SV4.2; no longer D12.C, R37.2, R58.1
- net N$66: now also R45.1, SV4.4; no longer R59.1
- net N$67: now also R57.1, R58.2; no longer R47.1, R60.2, SV4.2
- net N$75: now also R61.1, U$10.1; no longer R63.2, R64.1
- net N$76: now also R62.1, U$10.5; no longer R64.2, U2.2
- net N$77: now also R63.1, U$10.7; no longer R66.1, U$10.1
- net N$78: now also R64.1, U$10.9; no longer R67.1, U$10.5
- net N$79: now also R77.1, U3.1; no longer R68.1, U$10.7
- net N$8: now also R22.1, U$6.5; no longer JP1.TIP, R1.1
- net N$80: now also C33.1, C35.1, C41.+, C43.+, D15.1, D16.1, IC8.1, IC9.1, R72.2, X3.1; no longer R69.1, U$10.9
- net N$86: now also R67.2, SV5.3; no longer R70.2, SV5.1
- net N$87: now also R68.2, SV5.4; no longer R71.2, SV5.2
- net N$88: now also R69.2, SV5.5; no longer R72.2, SV5.3
- net N$89: now also R70.2, SV5.6; no longer R73.2, SV5.4
- net N$90: now also R71.2, SV5.8; no longer R74.2, SV5.5
- net N$95: now also JP6.TIP, R78.1; no longer JP5.TIP, R65.1
- net N$98: now also R74.2, R75.2, R76.2, R80.1; no longer JP6.TIP, R83.1
- net N$99: now also D17.C, R61.2, R83.1; no longer R86.1, TSOP2.OUT
- net RESET1: now also D11.C, R22.2, R49.1; no longer D10.C, R34.2, R52.1
- net RESET2: now also D18.C, R62.2, R79.1; no longer D16.C, R67.2, R84.1
- net RESET3: now also D25.C, R109.1, R92.2; no longer D22.C, R116.1, R99.2
- net SCK1: now also D12.C, R23.2; no longer D11.C, R36.2
- net SCK2: now also D19.C, R63.2; no longer D17.C, R68.2
- net SCK3: now also D26.C, R93.2; no longer D23.C, R100.2
- net SWITCH_DOWN1: now also R56.1; no longer R60.1
- net SWITCH_DOWN2: now also R86.1; no longer R92.1
- net SWITCH_DOWN3: now also R116.1; no longer R124.1
- net SWITCH_OK1: now also R58.1; no longer R62.1
- net SWITCH_OK2: now also R88.1; no longer R94.1
- net SWITCH_OK3: now also R118.1; no longer R126.1
- net SWITCH_UP1: now also R46.1; no longer R49.1
- net SWITCH_UP2: now also R76.1; no longer R81.1
- net SWITCH_UP3: now also R106.1; no longer R113.1
- net TSOP_OUT: now also D7.C, R40.2; no longer R22.2, R23.2
- net TSOP_OUT1: now also D14.C, R51.2; no longer R54.2, R56.2
- net TSOP_OUT2: now also D21.C, R81.2; no longer R86.2, R88.2
- net TSOP_OUT3: now also D28.C, R111.2; no longer R118.2, R120.2
Routing:
- net N$82 (its old number): track 68.1 -> 0.00 mm
- net N$120 (its old number): track 68.1 -> 0.00 mm
- net N$43 (its old number): track 68.1 -> 0.00 mm
- net N$42: track 3.40 -> 68.1 mm
- net N$117: track 9.14 -> 68.1 mm, vias 1 -> 0
- net N$80: track 10.5 -> 68.1 mm, vias 1 -> 0
- net N$64: track 38.1 -> 2.50 mm
- net N$123: track 0.00 -> 35.0 mm, vias 0 -> 1
- net N$128: track 31.0 -> 0.00 mm, vias 1 -> 0
- net N$99: track 7.48 -> 38.1 mm, vias 1 -> 0
- net N$140: track 38.1 -> 10.6 mm
- net N$84: track 0.00 -> 27.4 mm, vias 0 -> 1
- net N$47: track 0.00 -> 27.4 mm, vias 0 -> 1
- net N$121: track 0.00 -> 27.4 mm, vias 0 -> 1
- net N$62: track 13.6 -> 38.1 mm
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- added copper zone on layer 16, net N$102
- added copper zone on layer 1, net N$105
- added copper zone on layer 16, net N$117
- added copper zone on layer 16, net N$128
- added copper zone on layer 1, net N$133
- added copper zone on layer 1, net N$134
- added copper zone on layer 1, net N$139
- added copper zone on layer 16, net N$142
- added copper zone on layer 16, net N$42
- added copper zone on layer 16, net N$54
- added copper zone on layer 1, net N$59
- added copper zone on layer 1, net N$60
- added copper zone on layer 1, net N$65
- added copper zone on layer 16, net N$68
- added copper zone on layer 1, net N$80
- added copper zone on layer 1, net N$91
- added copper zone on layer 16, net N$96
- added copper zone on layer 16, net N$97
- removed copper zone on layer 16, net N$100
- removed copper zone on layer 16, net N$105
- removed copper zone on layer 1, net N$108 (its old number)
- removed copper zone on layer 16, net N$120 (its old number)
- removed copper zone on layer 16, net N$131 (its old number)
- removed copper zone on layer 1, net N$137
- removed copper zone on layer 1, net N$138
- removed copper zone on layer 1, net N$143 (its old number)
- removed copper zone on layer 16, net N$146 (its old number)
- removed copper zone on layer 16, net N$43 (its old number)
- removed copper zone on layer 16, net N$55 (its old number)
- removed copper zone on layer 1, net N$61
- removed copper zone on layer 1, net N$62
- removed copper zone on layer 1, net N$67
- removed copper zone on layer 16, net N$70 (its old number)
- removed copper zone on layer 1, net N$82 (its old number)
- removed copper zone on layer 1, net N$93 (its old number)
- removed copper zone on layer 16, net N$99
Other:
- board size 229.9 x 132 mm -> 229.9 x 130.7 mm
